File: kiCadFiles/miniShieldESP32.sch (KiCad schematic (older format))
At the start: 38 parts, among them J1 VIM, J2 OUT, J3 I2C, J4 I2C, J5 I2C, Q1 BC846, Q2 BC846, Q3 BC846, Q4 BC846, Q5 BC846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

Commit message: update
Parts:
- removed J1: VIM, MyFootprint:AK300-2, symbol Connector:Conn_01x02_Female
- removed J2: OUT, MyFootprint:AK300-2, symbol Connector:Conn_01x02_Female
- removed U1: ESP32-DEVKITC-32D, MyFootprint:MODULE_ESP32-DEVKITC-32D, symbol ESP32-DEVKITC-32D:ESP32-DEVKITC-32D
- added J1: VIM, MyFootprint:AK300-2, symbol Connector_Generic:Conn_01x02
- added J2: OUT, MyFootprint:AK300-2, symbol Connector_Generic:Conn_01x02
- added U1: ESP32-DEVKITC-32D-ESP32-DEVKITC-32D, MODULE_ESP32-DEVKITC-32D, symbol miniShieldESP32-rescue:ESP32-DEVKITC-32D-ESP32-DEVKITC-32D
Connections:
- net +3V3: now also U1.1 (3V3)
- net +5V: now also U1.19 (EXT_5V)
- net ADC1_CH3: now also U1.4 (SENSOR_VN)
- net ADC1_CH4: now also U1.7 (IO32)
- net ADC1_CH5: now also U1.8 (IO33)
- net ADC1_CH6: now also U1.5 (IO34)
- net ADC1_CH7: now also U1.6 (IO35)
- net Earth: now also J1.2 (Pin_2), U1.14 (GND1), U1.20 (GND3), U1.26 (GND2)
- net GPIO15: now also U1.35 (IO15)
- net GPIO16: now also U1.31 (IO16)
- net GPIO17: now also U1.30 (IO17)
- net GPIO18: now also U1.28 (IO18)
- net GPIO19: now also U1.27 (IO19)
- net GPIO2: now also U1.34 (IO2)
- net GPIO23: now also U1.21 (IO23)
- net GPIO25: now also U1.9 (IO25)
- net GPIO26: now also U1.10 (IO26)
- net GPIO27: now also U1.11 (IO27)
- net GPIO4: now also U1.32 (IO4)
- net GPIO5: now also U1.29 (IO5)
- net OUT1: now also J2.1 (Pin_1)
- net OUT2: now also J2.2 (Pin_2)
- net SCL: now also U1.22 (IO22)
- net SDA: now also U1.25 (IO21)
- net at D4.2 (A): now also J1.1 (Pin_1)
- new net GPIO13: U1.15 (IO13)
Other:
- note added: "IHM"
- note added: "M2M"
- note added: "MICRO"
- note added: "VIM"
- moved on the sheet: AFF1, D1, D2, D3, J3, J4, J5, Q1, Q2, Q3, Q4, Q5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

Commit message: arruamdno legendas, lesd e dht11
Parts:
- added R15: 10k, MyFootprint:Resistor_Vertical_RM3mm, symbol Device:R
Connections:
- net DHT11 is gone; now on net GPIO13: U2.2 (IO)
- net +3V3: now also D1.2 (A), D2.2 (A), D3.2 (A), R15.1; no longer D1.1 (K), D2.1 (K), D3.1 (K)
- net GPIO13: now also R15.2
- net at R1.1: now also D1.1 (K); no longer D1.2 (A)
- net at R2.1: now also D2.1 (K); no longer D2.2 (A)
- net at R3.1: now also D3.1 (K); no longer D3.2 (A)
Other:
- moved on the sheet: D1, D2, D3
Changed lines of the file:
@@
 Sheet 1 1
 Title ""
-Date "2021-03-10"
+Date "2021-03-11"
 Rev "REV 1.00"
 Comp "Shield IoT EDU-IFSP"
@@
 U 1 1 603ED9DF
 P 2850 1650
-F 0 "D1" V 2797 1730 50  0000 L CNN
-F 1 "LED_ALT" V 2888 1730 50  0000 L CNN
+F 0 "D1" V 2800 1750 50  0000 L CNN
+F 1 "LED_ALT" H 2650 1500 50  0000 L CNN
 F 2 "LED_THT:LED_D3.0mm" H 2850 1650 50  0001 C CNN
 F 3 "~" H 2850 1650 50  0001 C CNN
 	1    2850 1650
-	0    1    1    0
+	0    -1   -1   0
 $EndComp
 $Comp
@@
 P 3900 1650
 F 0 "D2" V 3847 1730 50  0000 L CNN
-F 1 "LED_ALT" V 3938 1730 50  0000 L CNN
+F 1 "LED_ALT" H 3700 1500 50  0000 L CNN
 F 2 "LED_THT:LED_D3.0mm" H 3900 1650 50  0001 C CNN
 F 3 "~" H 3900 1650 50  0001 C CNN
 	1    3900 1650
-	0    1    1    0
+	0    -1   -1   0
 $EndComp
 $Comp
@@
 P 4950 1650
 F 0 "D3" V 4897 1730 50  0000 L CNN
-F 1 "LED_ALT" V 4988 1730 50  0000 L CNN
+F 1 "LED_ALT" H 4750 1500 50  0000 L CNN
 F 2 "LED_THT:LED_D3.0mm" H 4950 1650 50  0001 C CNN
 F 3 "~" H 4950 1650 50  0001 C CNN
 	1    4950 1650
-	0    1    1    0
+	0    -1   -1   0
 $EndComp
 $Comp
@@
 $EndComp
 Wire Wire Line
-	10050 4650 10050 4900
+	10050 4650 10050 4700
 $Comp
 L power:Earth #PWR0108
@@
 Wire Wire Line
 	10050 6450 10050 5500
-Text Label 10550 5200 0    50   ~ 0
-DHT11
-Wire Wire Line
-	10550 5200 10350 5200
+Wire Wire Line
+	10550 5200 10400 5200
 $Comp
 L power:Earth #PWR0109
@@
 Wire Wire Line
 	1800 6400 2250 6400
-NoConn ~ 2250 6100
 NoConn ~ 2250 6200
 Connection ~ 3950 5600
@@
 F 3 "~" H 5950 2500 50  0001 C CNN
 	1    5950 2500
-	1    0    0    -1
-$EndComp
-$Comp
-L miniShieldESP32-rescue:ESP32-DEVKITC-32D-ESP32-DEVKITC-32D U1
-U 1 1 604A612D
-P 3050 5900
-F 0 "U1" H 3050 7067 50  0000 C CNN
-F 1 "ESP32-DEVKITC-32D-ESP32-DEVKITC-32D" H 3050 6976 50  0000 C CNN
-F 2 "MODULE_ESP32-DEVKITC-32D" H 3050 5900 50  0001 L BNN
-F 3 "" H 3050 5900 50  0001 L BNN
-F 4 "4" H 3050 5900 50  0001 L BNN "PARTREV"
-F 5 "Espressif Systems" H 3050 5900 50  0001 L BNN "MANUFACTURER"
-	1    3050 5900
 	1    0    0    -1
 $EndComp
@@
 Text Notes 1350 4250 0    67   ~ 13
 MICRO
+$Comp
+L miniShieldESP32-rescue:ESP32-DEVKITC-32D-ESP32-DEVKITC-32D U1
+U 1 1 604A612D
+P 3050 5900
+F 0 "U1" H 3050 7067 50  0000 C CNN
+F 1 "ESP32-DEVKITC-32D-ESP32-DEVKITC-32D" H 3050 6976 50  0000 C CNN
+F 2 "MODULE_ESP32-DEVKITC-32D" H 3050 5900 50  0001 L BNN
+F 3 "" H 3050 5900 50  0001 L BNN
+F 4 "4" H 3050 5900 50  0001 L BNN "PARTREV"
+F 5 "Espressif Systems" H 3050 5900 50  0001 L BNN "MANUFACTURER"
+	1    3050 5900
+	1    0    0    -1
+$EndComp
+NoConn ~ 2250 6100
+Text Label 10550 5200 0    50   ~ 0
+GPIO13
+Wire Wire Line
+	10400 5050 10400 5200
+Connection ~ 10400 5200
+Wire Wire Line
+	10400 5200 10350 5200
+Wire Wire Line
+	10400 4750 10400 4700
+Wire Wire Line
+	10400 4700 10050 4700
+Connection ~ 10050 4700
+Wire Wire Line
+	10050 4700 10050 4900
+$Comp
+L Device:R R15
+U 1 1 60802690
+P 10400 4900
+F 0 "R15" H 10470 4946 50  0000 L CNN
+F 1 "10k" V 10400 4800 50  0000 L CNN
+F 2 "MyFootprint:Resistor_Vertical_RM3mm" V 10330 4900 50  0001 C CNN
+F 3 "~" H 10400 4900 50  0001 C CNN
+	1    10400 4900
+	1    0    0    -1
+$EndComp
 $EndSCHEMATC
