File: kiCadFiles/miniShieldESP32.kicad_pcb (KiCad board)
At the start: 2 copper layers, 92 x 61 mm, 42 parts, among them J1 VIM, J2 OUT, J3 I2C, J4 I2C, J5 I2C, Q1 BC846, Q2 BC846, Q3 BC846, Q4 BC846, Q5 BC846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

Commit message: arruamdno legendas, lesd e dht11
Parts:
- added R15: 10k, MyFootprint:Resistor_Vertical_RM3mm, F.Cu at (158.9, 55.4)
- U1: value ESP32-DEVKITC-32D -> ESP32-DEVKITC-32D-ESP32-DEVKITC-32D
- moved REF** 25.1 mm to (137.4, 58.3)
- moved REF** 23.8 mm to (133.8, 69.7)
- moved D1 2.72 mm to (175.9, 63.0), turned to 0 degrees
- moved D2 2.72 mm to (175.9, 57.0), turned to 0 degrees
- moved D3 2.72 mm to (175.9, 51.0), turned to 0 degrees
- moved G*** 2.23 mm to (166.8, 87.0)
- moved J2 0.07 mm to (111.9, 52.3)
- moved J1 0.05 mm to (101.7, 52.3)
Connections:
- net /DHT11 renamed /GPIO13
- D1 pad 1: +3V3 -> Net-(D1-Pad1)
- D1 pad 2: Net-(D1-Pad2) -> +3V3
- D2 pad 1: +3V3 -> Net-(D2-Pad1)
- D2 pad 2: Net-(D2-Pad2) -> +3V3
- D3 pad 1: +3V3 -> Net-(D3-Pad1)
- D3 pad 2: Net-(D3-Pad2) -> +3V3
- R1 pad 1: Net-(D1-Pad2) -> Net-(D1-Pad1)
- R2 pad 1: Net-(D2-Pad2) -> Net-(D2-Pad1)
- R3 pad 1: Net-(D3-Pad2) -> Net-(D3-Pad1)
Routing:
- net +3V3: track 216.5 -> 224.1 mm
- net Net-(D2-Pad2): track 4.04 -> 0.00 mm
- net Net-(D2-Pad1): track 0.00 -> 4.04 mm
- net Net-(D1-Pad2): track 4.04 -> 0.00 mm
- net Net-(D1-Pad1): track 0.00 -> 4.04 mm
- net Net-(D3-Pad2): track 4.04 -> 0.00 mm
- net Net-(D3-Pad1): track 0.00 -> 4.04 mm
- net /GPIO13: track 17.5 -> 16.0 mm
Other:
- board text added: "-"
- board text added: "A-GPIO04"
- board text added: "ADC1_CH3 - GPIO27"
- board text added: "ADC1_CH6 GPIO34"
- board text added: "B-GPIO16"
- board text added: "C-GPIO23"
- board text added: "D-GPIO19"
- board text added: "E-GPIO18"
- board text added: "F-GPIO17"
- board text added: "G-GPIO05"
- board text added: "GPIO13"
- board text added: "GPIO25"
- board text added: "GPIO26"
- board text added: "GPIO27"
- board text added: "GPIO32"
- board text added: "GPIO33"
- board text added: "GPIO35"
- board text added: "OUT1GPIO02"
- board text added: "OUT1GPIO15"
- board text added: "SCL"
- board text added: "SCL-GPIO22"
- board text added: "SDA"
- board text added: "SDA-GPIO21"

Commit message: gerber
Parts:
- removed the REF** at (137.4, 58.3)
- removed the REF** at (133.8, 69.7)
- added REF**: MountingHole_3.2mm_M3, MountingHole:MountingHole_3.2mm_M3, F.Cu at (146.8, 100.5)
- added REF**: MountingHole_3.2mm_M3, MountingHole:MountingHole_3.2mm_M3, F.Cu at (127.8, 54.5)
